File: dev_interface.kicad_sch (KiCad schematic)
At the start: 17 parts, among them U10 ADS1014IDGS, U11 ADS1014IDGS, U4 ISO164xB, U5 DACx53401, U6 DACx53401, U8 LM2904

Commit message: Fix ground references
Connections:
- net GND: no longer C16.1, U10.5 (AIN1), U11.5 (AIN1), U8.4 (V-)
- new net GNDPWR: C16.1, U10.5 (AIN1), U11.5 (AIN1), U8.4 (V-)

Commit message: last formatting change I promise
Connections:
- net SCL_{INT}: now also U4.6 (SCL2); no longer U4.7 (SDA2)
- net SDA_{INT}: now also U4.7 (SDA2); no longer U4.6 (SCL2)
Other:
- moved on the sheet: C10, C11, C12, C13, C14, C15, C16, C17, C18, R10, R11, U10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

Commit message: formatting!?!? idk what I changed tbh
Parts:
- added R22, R23: 1.5k, Resistor_SMD:R_0603_1608Metric_Pad0.98x0.95mm_HandSolder, symbol Device:R
Connections:
- net +3V3: now also U5.7 (FB), U6.7 (FB), R22.1, R23.1; no longer C16.2, U5.6 (VDD), U6.6 (VDD), U8.8 (V+)
- net DAC_{1}_FB: now also U5.5 (AGND); no longer U5.7 (FB)
- net DAC_{2}_FB: now also U6.5 (AGND); no longer U6.7 (FB)
- net GND: now also U5.8 (OUT), U6.8 (OUT); no longer U5.5 (AGND), U6.5 (AGND)
- net POW_DRAW: now also U6.6 (VDD); no longer U6.8 (OUT)
- net POW_LIMIT: now also U5.6 (VDD); no longer U5.8 (OUT)
- net SCL_{INT}: now also R22.2
- net SDA_{INT}: now also R23.2
- new net +24V: C16.2, U8.8 (V+)
Other:
- title: (none) -> Dev Board Interface
- moved on the sheet: C12, C13, C14, C15, C16, C18, U10, U11, U8B, U8C

Commit message: Update library + update symbols
Connections:
- net +3V3: now also U5.6 (VDD), U6.6 (VDD); no longer U5.7 (FB), U6.7 (FB)
- net DAC_{1}_FB: now also U5.7 (FB); no longer U5.5 (AGND)
- net DAC_{2}_FB: now also U6.7 (FB); no longer U6.5 (AGND)
- net GND: now also U5.5 (AGND), U6.5 (AGND); no longer U5.8 (OUT), U6.8 (OUT)
- net POW_DRAW: now also U6.8 (OUT); no longer U6.6 (VDD)
- net POW_LIMIT: now also U5.8 (OUT); no longer U5.6 (VDD)

Commit message: Updating symbol library + passing some ERC tests
Parts:
- U7: renamed from U4; symbol ! Robomaster:ISO164xB -> ! Robomaster ICs:ISO164xB
- U8: renamed from U5; symbol ! Robomaster:DACx3401 -> ! Robomaster ICs:DACx3401
- U9: renamed from U6; symbol ! Robomaster:DACx3401 -> ! Robomaster ICs:DACx3401
- renumbered C14 to C10, C15 to C11, C16 to C3, C17 to C4, C18 to C5, C11 to C6, C13 to C7, C12 to C8, C10 to C9, R22 to R17, R23 to R18, R10 to R19, R11 to R20, U8 to U3, U10 to U5, U11 to U6

Commit message: Add input resistor divider to battery voltage ADC
+ renumbered components
Parts:
- added R11: 180k, Resistor_SMD:R_0603_1608Metric_Pad0.98x0.95mm_HandSolder, symbol Device:R
- added R12: 120k, Resistor_SMD:R_0603_1608Metric_Pad0.98x0.95mm_HandSolder, symbol Device:R
- renumbered C11 to C10, C3 to C2, C4 to C3, C5 to C4, C6 to C5, C7 to C6, C8 to C7, C9 to C8, C10 to C9, R17 to R13, R18 to R14, R19 to R15, R20 to R16, U3 to U2, U5 to U4, U6 to U5, U7 to U6, U8 to U7, U9 to U8
Connections:
- net GND: now also R12.2
- net V_{SC}: now also R11.1; no longer U2.5 (+)
- new net V_{SC}_scaled: R11.2, R12.1, U2.5 (+)

Commit message: Add in voltage control for components
Other:
- note added: "Input scaling: 180k over 120k = ^{2}/_{5}"
Changed lines of the file:
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@@
 	(wire
 		(pts
-			(xy 207.01 57.15) (xy 207.01 54.61)
+			(xy 241.3 57.15) (xy 241.3 54.61)
 		)
 		(stroke
@@
 	(wire
 		(pts
-			(xy 207.01 54.61) (xy 204.47 54.61)
+			(xy 241.3 54.61) (xy 204.47 54.61)
 		)
 		(stroke
@@
 		)
 	)
+	(text "Input scaling:\n180k over 120k = ^{2}/_{5}"
+		(exclude_from_sim no)
+		(at 56.896 143.256 0)
+		(effects
+			(font
+				(size 1.27 1.27)
+			)
+		)
+	)
 	(text "DAC_{2} ADDR:\n1001000R_{2}"
 		(exclude_from_sim no)
@@
 	(symbol
 		(lib_id "power:GNDD")
-		(at 207.01 57.15 0)
+		(at 241.3 57.15 0)
 		(unit 1)
 		(exclude_from_sim no)
@@
 		(fields_autoplaced yes)
 		(property "Reference" "#PWR038"
-			(at 207.01 63.5 0)
+			(at 241.3 63.5 0)
 			(effects
 				(font
@@
 		)
 		(property "Value" "GNDD"
-			(at 207.01 60.96 0)
+			(at 241.3 60.96 0)
 			(effects
 				(font
@@
 		)
 		(property "Footprint" ""
-			(at 207.01 57.15 0)
+			(at 241.3 57.15 0)
 			(effects
 				(font
@@
 		)
 		(property "Datasheet" ""
-			(at 207.01 57.15 0)
+			(at 241.3 57.15 0)
 			(effects
 				(font
@@
 		)
 		(property "Description" "Power symbol creates a global label with name \"GNDD\" , digital ground"
-			(at 207.01 57.15 0)
+			(at 241.3 57.15 0)
 			(effects
 				(font

Commit message: Finish up buck
Parts:
- C10, C2, C3, C4, C9: footprint (none) -> Capacitor_SMD:C_0603_1608Metric_Pad1.08x0.95mm_HandSolder
Changed lines of the file:
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@@
 			)
 		)
-		(property "Footprint" ""
+		(property "Footprint" "Capacitor_SMD:C_0603_1608Metric_Pad1.08x0.95mm_HandSolder"
 			(at 68.2752 91.44 0)
 			(effects
@@
 			)
 		)
-		(property "Footprint" ""
+		(property "Footprint" "Capacitor_SMD:C_0603_1608Metric_Pad1.08x0.95mm_HandSolder"
 			(at 225.0948 132.08 0)
 			(effects
@@
 			)
 		)
-		(property "Footprint" ""
+		(property "Footprint" "Capacitor_SMD:C_0603_1608Metric_Pad1.08x0.95mm_HandSolder"
 			(at 127 120.3452 0)
 			(effects
@@
 			)
 		)
-		(property "Footprint" ""
+		(property "Footprint" "Capacitor_SMD:C_0603_1608Metric_Pad1.08x0.95mm_HandSolder"
 			(at 225.0948 101.6 0)
 			(effects
@@
 			)
 		)
-		(property "Footprint" ""
+		(property "Footprint" "Capacitor_SMD:C_0603_1608Metric_Pad1.08x0.95mm_HandSolder"
 			(at 127 75.8952 0)
 			(effects
