File: ideal_diode.kicad_sch (KiCad schematic)
At the start: 8 parts, among them Q1 Q_NMOS_DSG, U12 SN74LVC2G08, U9 LTC4357DCB

Commit message: Added proper peripherals to ideal diode controller
also updated library
Parts:
- removed R17: 100, Resistor_SMD:R_0603_1608Metric_Pad0.98x0.95mm_HandSolder, symbol Device:R
- removed U9: LTC4357DCB, Package_DFN_QFN:DFN-6-1EP_3x2mm_P0.5mm_EP1.65x1.35mm, symbol Power_Management:LTC4357DCB
- added C25: 0.1u, Capacitor_SMD:C_0603_1608Metric_Pad1.08x0.95mm_HandSolder, symbol Device:C
- added C26: 0.022u, Capacitor_SMD:C_0603_1608Metric_Pad1.08x0.95mm_HandSolder, symbol Device:C
- added D1: SMBJ26A, Diode_SMD:D_SMB_Handsoldering, symbol Device:D_Zener
- added D2: SMBJ58A, Diode_SMD:D_SMB_Handsoldering, symbol Device:D_Zener
- added U14: LM74700, Package_TO_SOT_SMD:SOT-23-6_Handsoldering, symbol Power_Management:LM74700
- C11: value 0.1u -> 47u
Connections:
- net OUT_{LPF} is gone; now on net OUT: C11.1
- net DIRECT_EN: now also U14.3 (EN)
- net GATE: now also U14.5 (GATE)
- net GNDPWR: now also C26.2, D1.1 (K), U14.2 (GND)
- net IN: now also C25.1, C26.1, D2.1 (K), U14.6 (ANODE)
- net OUT: now also U14.4 (CATHODE)
- new net TVS_mid: D1.2 (A), D2.2 (A)
- new net VCAP: C25.2, U14.1 (VCAP)

Commit message: Polish up ideal diode subsheet
Made custom symbol for multipinned FET
Parts:
- Q1: value Q_NMOS_DSG -> NVMFS5C404NL; footprint (none) -> Package_SO:ONSemi_SO-8FL_488AA; symbol Device:Q_NMOS_DSG -> Device:Q_NMOS_SGD
Connections:
- net GATE: now also Q1.4 (G); no longer Q1.3 (G)
- net IN: now also Q1.5 (D); no longer Q1.1 (D)
- net OUT: now also Q1.1 (S), Q1.3 (S)
Other:
- title: (none) -> Ideal Diode + VSense
Changed lines of the file:
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@@
 	(paper "A4")
 	(title_block
+		(title "Ideal Diode + VSense")
 		(date "2024-12-06")
 		(rev "1")
@@
 	)
 	(junction
+		(at 161.29 48.26)
+		(diameter 0)
+		(color 0 0 0 0)
+	)
+	(junction
 		(at 124.46 71.12)
 		(diameter 0)
@@
 	)
 	(junction
+		(at 161.29 45.72)
+		(diameter 0)
+		(color 0 0 0 0)
+	)
+	(junction
 		(at 162.56 48.26)
 		(diameter 0)
@@
 	(wire
 		(pts
+			(xy 161.29 45.72) (xy 161.29 48.26)
+		)
+		(stroke
+			(width 0)
+			(type default)
+		)
+	)
+	(wire
+		(pts
 			(xy 124.46 58.42) (xy 124.46 71.12)
 		)
@@
 	(wire
 		(pts
-			(xy 160.02 48.26) (xy 162.56 48.26)
+			(xy 161.29 43.18) (xy 161.29 45.72)
+		)
+		(stroke
+			(width 0)
+			(type default)
+		)
+	)
+	(wire
+		(pts
+			(xy 160.02 48.26) (xy 161.29 48.26)
 		)
 		(stroke
@@
 	(wire
 		(pts
+			(xy 160.02 43.18) (xy 161.29 43.18)
+		)
+		(stroke
+			(width 0)
+			(type default)
+		)
+	)
+	(wire
+		(pts
 			(xy 124.46 71.12) (xy 124.46 82.55)
 		)
@@
 	(wire
 		(pts
+			(xy 160.02 45.72) (xy 161.29 45.72)
+		)
+		(stroke
+			(width 0)
+			(type default)
+		)
+	)
+	(wire
+		(pts
 			(xy 186.69 129.54) (xy 186.69 130.81)
+		)
+		(stroke
+			(width 0)
+			(type default)
+		)
+	)
+	(wire
+		(pts
+			(xy 161.29 48.26) (xy 162.56 48.26)
 		)
 		(stroke
@@
 	)
 	(symbol
-		(lib_id "Device:Q_NMOS_DSG")
+		(lib_id "Device:Q_NMOS_SGD")
 		(at 154.94 50.8 90)
 		(unit 1)
@@
 		(on_board yes)
 		(dnp no)
-		(fields_autoplaced yes)
 		(property "Reference" "Q1"
 			(at 154.94 41.91 90)
@@
 			)
 		)
-		(property "Value" "Q_NMOS_DSG"
-			(at 154.94 44.45 90)
-			(effects
-				(font
-					(size 1.27 1.27)
-				)
-			)
-		)
-		(property "Footprint" ""
+		(property "Value" "NVMFS5C404NL"
+			(at 149.352 44.196 90)
+			(effects
+				(font
+					(size 1.27 1.27)
+				)
+			)
+		)
+		(property "Footprint" "Package_SO:ONSemi_SO-8FL_488AA"
 			(at 152.4 45.72 0)
 			(effects
@@
 			)
 		)
-		(property "Description" "N-MOSFET transistor, drain/source/gate"
+		(property "Description" "N-MOSFET transistor, source/gate/drain"
 			(at 154.94 50.8 0)
 			(effects
@@
 		(pin "3"
 		)
+		(pin "4"
+		)
+		(pin "5"
+		)
 		(instances

Commit message: Reannotated
Parts:
- renumbered C26 to C24, C11 to C26, C20 to C27, D2 to D4, D1 to D5, Q1 to Q3, U12 to U10, U14 to U11
Changed lines of the file:
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@@
 		(on_board yes)
 		(dnp no)
-		(property "Reference" "C11"
+		(property "Reference" "C26"
 			(at 172.72 53.3399 0)
 			(effects
@@
 			(project "SupercapManager"
 				(path "/6197145b-e7d4-44cc-9d90-537b6501bf60/f28a7bbd-a217-4ab0-a73c-be6ca56ea928"
-					(reference "C11")
+					(reference "C26")
 					(unit 1)
 				)
@@
 		(on_board yes)
 		(dnp no)
-		(property "Reference" "C26"
+		(property "Reference" "C24"
 			(at 120.65 53.3399 0)
 			(effects
@@
 			(project "SupercapManager"
 				(path "/6197145b-e7d4-44cc-9d90-537b6501bf60/f28a7bbd-a217-4ab0-a73c-be6ca56ea928"
-					(reference "C26")
+					(reference "C24")
 					(unit 1)
 				)
@@
 		(dnp no)
 		(fields_autoplaced yes)
-		(property "Reference" "#PWR051"
+		(property "Reference" "#PWR058"
 			(at 88.9 109.22 0)
 			(effects
@@
 			(project ""
 				(path "/6197145b-e7d4-44cc-9d90-537b6501bf60/f28a7bbd-a217-4ab0-a73c-be6ca56ea928"
-					(reference "#PWR051")
+					(reference "#PWR058")
 					(unit 1)
 				)
@@
 		(dnp no)
 		(fields_autoplaced yes)
-		(property "Reference" "U12"
+		(property "Reference" "U10"
 			(at 129.5289 118.11 0)
 			(effects
@@
 			(project ""
 				(path "/6197145b-e7d4-44cc-9d90-537b6501bf60/f28a7bbd-a217-4ab0-a73c-be6ca56ea928"
-					(reference "U12")
+					(reference "U10")
 					(unit 2)
 				)
@@
 		(dnp no)
 		(fields_autoplaced yes)
-		(property "Reference" "#PWR049"
+		(property "Reference" "#PWR063"
 			(at 186.69 135.89 0)
 			(effects
@@
 			(project "SupercapManager"
 				(path "/6197145b-e7d4-44cc-9d90-537b6501bf60/f28a7bbd-a217-4ab0-a73c-be6ca56ea928"
-					(reference "#PWR049")
+					(reference "#PWR063")
 					(unit 1)
 				)
@@
 		(dnp no)
 		(fields_autoplaced yes)
-		(property "Reference" "#PWR050"
+		(property "Reference" "#PWR062"
 			(at 186.69 109.22 0)
 			(effects
@@
 			(project "SupercapManager"
 				(path "/6197145b-e7d4-44cc-9d90-537b6501bf60/f28a7bbd-a217-4ab0-a73c-be6ca56ea928"
-					(reference "#PWR050")
+					(reference "#PWR062")
 					(unit 1)
 				)
@@
 		(dnp no)
 		(fields_autoplaced yes)
-		(property "Reference" "#PWR044"
+		(property "Reference" "#PWR060"
 			(at 124.46 88.9 0)
 			(effects
@@
 			(project "SupercapManager"
 				(path "/6197145b-e7d4-44cc-9d90-537b6501bf60/f28a7bbd-a217-4ab0-a73c-be6ca56ea928"
-					(reference "#PWR044")
+					(reference "#PWR060")
 					(unit 1)
 				)
@@
 		(on_board yes)
 		(dnp no)
-		(property "Reference" "Q1"
+		(property "Reference" "Q3"
 			(at 154.94 41.91 90)
 			(effects
@@
 			(project "SupercapManager"
 				(path "/6197145b-e7d4-44cc-9d90-537b6501bf60/f28a7bbd-a217-4ab0-a73c-be6ca56ea928"
-					(reference "Q1")
+					(reference "Q3")
 					(unit 1)
 				)
@@
 		(dnp no)
 		(fields_autoplaced yes)
-		(property "Reference" "U14"
+		(property "Reference" "U11"
 			(at 166.37 68.5799 0)
 			(effects
@@
 			(project ""
 				(path "/6197145b-e7d4-44cc-9d90-537b6501bf60/f28a7bbd-a217-4ab0-a73c-be6ca56ea928"
-					(reference "U14")
+					(reference "U11")
 					(unit 1)
 				)
@@
 		(dnp no)
 		(fields_autoplaced yes)
-		(property "Reference" "U12"
+		(property "Reference" "U10"
 			(at 193.04 116.8399 0)
 			(effects
@@
 			(project ""
 				(path "/6197145b-e7d4-44cc-9d90-537b6501bf60/f28a7bbd-a217-4ab0-a73c-be6ca56ea928"
-					(reference "U12")
+					(reference "U10")
 					(unit 3)
 				)
@@
 		(on_board yes)
 		(dnp no)
-		(property "Reference" "D2"
+		(property "Reference" "D4"
 			(at 106.68 53.3399 90)
 			(effects
@@
 			(project "SupercapManager"
 				(path "/6197145b-e7d4-44cc-9d90-537b6501bf60/f28a7bbd-a217-4ab0-a73c-be6ca56ea928"
-					(reference "D2")
+					(reference "D4")
 					(unit 1)
 				)
@@
 		(dnp no)
 		(fields_autoplaced yes)
-		(property "Reference" "#PWR08"
+		(property "Reference" "#PWR061"
 			(at 176.53 66.04 0)
 			(effects
@@
 			(project "SupercapManager"
 				(path "/6197145b-e7d4-44cc-9d90-537b6501bf60/f28a7bbd-a217-4ab0-a73c-be6ca56ea928"
-					(reference "#PWR08")
+					(reference "#PWR061")
 					(unit 1)
 				)
@@
 		(on_board yes)
 		(dnp no)
-		(property "Reference" "C20"
+		(property "Reference" "C27"
 			(at 173.99 116.8399 0)
 			(effects
@@
 			(project "SupercapManager"
 				(path "/6197145b-e7d4-44cc-9d90-537b6501bf60/f28a7bbd-a217-4ab0-a73c-be6ca56ea928"
-					(reference "C20")
+					(reference "C27")
 					(unit 1)
 				)
@@
 		(dnp no)
 		(fields_autoplaced yes)
-		(property "Reference" "U12"
+		(property "Reference" "U10"
 			(at 129.5289 99.06 0)
 			(effects
@@
 			(project ""
 				(path "/6197145b-e7d4-44cc-9d90-537b6501bf60/f28a7bbd-a217-4ab0-a73c-be6ca56ea928"
-					(reference "U12")
+					(reference "U10")
 					(unit 1)
 				)
@@
 		(dnp no)
 		(fields_autoplaced yes)
-		(property "Reference" "#PWR052"
+		(property "Reference" "#PWR059"
 			(at 88.9 138.43 0)
 			(effects
@@
 			(project "SupercapManager"
 				(path "/6197145b-e7d4-44cc-9d90-537b6501bf60/f28a7bbd-a217-4ab0-a73c-be6ca56ea928"
-					(reference "#PWR052")
+					(reference "#PWR059")
 					(unit 1)
 				)
@@
 		(on_board yes)
 		(dnp no)
-		(property "Reference" "D1"
+		(property "Reference" "D5"
 			(at 106.68 63.4999 90)
 			(effects
@@
 			(project ""
 				(path "/6197145b-e7d4-44cc-9d90-537b6501bf60/f28a7bbd-a217-4ab0-a73c-be6ca56ea928"
-					(reference "D1")
-					(unit 1)
-				)
+					(reference "D5")
+					(unit 1)
+				)

Commit message: Attempting to use just an opamp probably won't work
Will use diff amp + schmitt trigger
Connections:
- net +24V is gone; now on net IN: R26.1
Changed lines of the file:
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@@
+	(wire
+		(pts
+			(xy 86.36 105.41) (xy 88.9 105.41)
+		)
+		(stroke
+			(width 0)
+			(type default)
+		)
+	)
 	(wire
 		(pts
@@
 		)
 	)
+	(hierarchical_label "IN"
+		(shape input)
+		(at 86.36 105.41 180)
+		(fields_autoplaced yes)
+		(effects
+			(font
+				(size 1.27 1.27)
+			)
+			(justify right)
+		)
+	)
 	(hierarchical_label "OUT"
 		(shape output)
@@
 					(unit 1)
 				)
-			)
-		)
-	)
-	(symbol
-		(lib_id "power:+24V")
-		(at 88.9 105.41 0)
-		(unit 1)
-		(exclude_from_sim no)
-		(in_bom yes)
-		(on_board yes)
-		(dnp no)
-		(fields_autoplaced yes)
-		(property "Reference" "#PWR058"
-			(at 88.9 109.22 0)
-			(effects
-				(font
-					(size 1.27 1.27)
-				)
-				(hide yes)
-			)
-		)
-		(property "Value" "+24V"
-			(at 88.9 100.33 0)
-			(effects
-				(font
-					(size 1.27 1.27)
-				)
-			)
-		)
-		(property "Footprint" ""
-			(at 88.9 105.41 0)
-			(effects
-				(font
-					(size 1.27 1.27)
-				)
-				(hide yes)
-			)
-		)
-		(property "Datasheet" ""
-			(at 88.9 105.41 0)
-			(effects
-				(font
-					(size 1.27 1.27)
-				)
-				(hide yes)
-			)
-		)
-		(property "Description" "Power symbol creates a global label with name \"+24V\""
-			(at 88.9 105.41 0)
-			(effects
-				(font
-					(size 1.27 1.27)
-				)
-				(hide yes)
-			)
-		)
-		(pin "1"
-		)
-		(instances
-			(project ""
-				(path "/6197145b-e7d4-44cc-9d90-537b6501bf60/f28a7bbd-a217-4ab0-a73c-be6ca56ea928"
-					(reference "#PWR058")
-					(unit 1)
-				)

Commit message: Ideating for diff amp
Parts:
- added D7: D, symbol Device:D
- added R40: R, symbol Device:R
Connections:
- net DIRECT_IEN: now also R40.1; no longer U10.1
- net GNDPWR: now also D7.2 (A)
- new net: D7.1 (K), R40.2, U10.1
Other:
- moved on the sheet: C27, U10A, U10B, U10C
