File: housekeeping.kicad_sch (KiCad schematic)
At the start: 44 parts, among them U14 MC34063A, U15 MC34063A, U16 TPS54302

Commit message: Unsure of changes
Parts:
- gave numbers to parts that had none: 3
- renumbered C51 to C14, C52 to C15, C53 to C16, C54 to C17, C55 to C18, C56 to C19, C57 to C20, C58 to C21, C59 to C22, C60 to C23, C61 to C24, C62 to C25, C63 to C26, C64 to C27, C65 to C28, C66 to C29, C67 to C30, C68 to C31, C69 to C32, C70 to C33, D6 to D2, D7 to D3, L4 to L1, L5 to L2, L6 to L3, R63 to R25, R64 to R26, R65 to R27, R66 to R28, R67 to R29, R68 to R30, R69 to R31, R70 to R32, R71 to R33, R72 to R34, R73 to R35, TP1 to TP5, TP2 to TP8, U14 to U11, U15 to U12, U16 to U13
Changed lines of the file:
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@@
 		(dnp no)
 		(fields_autoplaced yes)
-		(property "Reference" "#PWR096"
+		(property "Reference" "#PWR093"
 			(at 104.14 167.64 0)
 			(effects
@@
 		(dnp no)
 		(fields_autoplaced yes)
-		(property "Reference" "#PWR085"
+		(property "Reference" "#PWR082"
 			(at 130.81 69.85 0)
 			(effects
@@
 		(on_board yes)
 		(dnp no)
-		(property "Reference" "R66"
+		(property "Reference" "R28"
 			(at 93.98 66.04 90)
 			(effects
@@
 		(on_board yes)
 		(dnp no)
-		(property "Reference" "C60"
+		(property "Reference" "C23"
 			(at 243.84 77.4699 0)
 			(effects
@@
 		(on_board yes)
 		(dnp no)
-		(property "Reference" "D6"
+		(property "Reference" "D2"
 			(at 231.14 48.5776 90)
 			(effects
@@
 		(dnp no)
 		(fields_autoplaced yes)
-		(property "Reference" "#PWR090"
+		(property "Reference" "#PWR087"
 			(at 184.15 88.9 0)
 			(effects
@@
 		(dnp no)
 		(fields_autoplaced yes)
-		(property "Reference" "L6"
+		(property "Reference" "L3"
 			(at 93.98 134.62 90)
 			(effects
@@
 		(dnp no)
 		(fields_autoplaced yes)
-		(property "Reference" "#PWR091"
+		(property "Reference" "#PWR088"
 			(at 116.84 91.44 0)
 			(effects
@@
 		(on_board yes)
 		(dnp no)
-		(property "Reference" "C61"
+		(property "Reference" "C24"
 			(at 255.27 77.4699 0)
 			(effects
@@
 		(dnp yes)
 		(fields_autoplaced yes)
-		(property "Reference" "TP?"
+		(property "Reference" "TP7"
 			(at 236.22 32.2579 0)
 			(effects
@@
 		)
 		(instances
-			(project "SupercapManager"
-				(path "/6197145b-e7d4-44cc-9d90-537b6501bf60/2b4de7d2-e111-42d9-afee-f810f96a2f61"
-					(reference "TP?")
-					(unit 1)
-				)
-			)
 			(project "Rev 1B"
 				(path "/e5f99deb-ef42-4c5f-b80a-388477910e20/1e0b2151-e075-4f05-b22a-12d6722ef31a"
@@
 		(dnp no)
 		(fields_autoplaced yes)
-		(property "Reference" "R73"
+		(property "Reference" "R35"
 			(at 106.68 154.9399 0)
 			(effects
@@
 		(on_board yes)
 		(dnp no)
-		(property "Reference" "R64"
+		(property "Reference" "R26"
 			(at 55.88 52.0701 0)
 			(effects
@@
 		(on_board yes)
 		(dnp no)
-		(property "Reference" "C70"
+		(property "Reference" "C33"
 			(at 134.62 144.272 90)
 			(effects
@@
 		(dnp yes)
 		(fields_autoplaced yes)
-		(property "Reference" "TP?"
+		(property "Reference" "TP6"
 			(at 175.26 32.2579 0)
 			(effects
@@
 		)
 		(instances
-			(project "SupercapManager"
-				(path "/6197145b-e7d4-44cc-9d90-537b6501bf60/2b4de7d2-e111-42d9-afee-f810f96a2f61"
-					(reference "TP?")
-					(unit 1)
-				)
-			)
 			(project "Rev 1B"
 				(path "/e5f99deb-ef42-4c5f-b80a-388477910e20/1e0b2151-e075-4f05-b22a-12d6722ef31a"
@@
 		(on_board yes)
 		(dnp no)
-		(property "Reference" "C62"
+		(property "Reference" "C25"
 			(at 166.37 116.4081 0)
 			(effects
@@
 		(dnp no)
 		(fields_autoplaced yes)
-		(property "Reference" "#PWR094"
+		(property "Reference" "#PWR091"
 			(at 50.8 153.67 0)
 			(effects
@@
 		(on_board yes)
 		(dnp no)
-		(property "Reference" "C69"
+		(property "Reference" "C32"
 			(at 129.54 144.272 90)
 			(effects
@@
 		(on_board yes)
 		(dnp no)
-		(property "Reference" "C56"
+		(property "Reference" "C19"
 			(at 207.01 79.502 90)
 			(effects
@@
 		(dnp no)
 		(fields_autoplaced yes)
-		(property "Reference" "#PWR084"
+		(property "Reference" "#PWR081"
 			(at 223.52 71.12 0)
 			(effects
@@
 		(dnp no)
 		(fields_autoplaced yes)
-		(property "Reference" "R72"
+		(property "Reference" "R34"
 			(at 106.68 143.5099 0)
 			(effects
@@
 		(dnp no)
 		(fields_autoplaced yes)
-		(property "Reference" "U15"
+		(property "Reference" "U12"
 			(at 196.85 40.64 0)
 			(effects
@@
 		(dnp yes)
 		(fields_autoplaced yes)
-		(property "Reference" "TP1"
+		(property "Reference" "TP5"
 			(at 96.52 35.5599 90)
 			(effects
@@
 		(on_board yes)
 		(dnp no)
-		(property "Reference" "R67"
+		(property "Reference" "R29"
 			(at 207.01 67.31 90)
 			(effects
@@
 		(on_board yes)
 		(dnp no)
-		(property "Reference" "D7"
+		(property "Reference" "D3"
 			(at 106.68 55.5624 90)
 			(effects
@@
 		(dnp no)
 		(fields_autoplaced yes)
-		(property "Reference" "#PWR092"
+		(property "Reference" "#PWR089"
 			(at 251.46 93.98 0)
 			(effects
@@
 		(dnp no)
 		(fields_autoplaced yes)
-		(property "Reference" "#PWR095"
+		(property "Reference" "#PWR092"
 			(at 115.57 161.29 0)
 			(effects
@@
 		(on_board yes)
 		(dnp no)
-		(property "Reference" "C51"
+		(property "Reference" "C14"
 			(at 95.25 55.88 0)
 			(effects
@@
 		(on_board yes)
 		(dnp no)
-		(property "Reference" "C66"
+		(property "Reference" "C29"
 			(at 114.3 144.272 90)
 			(effects
@@
 		(dnp no)
 		(fields_autoplaced yes)
-		(property "Reference" "#PWR088"
+		(property "Reference" "#PWR085"
 			(at 170.18 74.93 0)
 			(effects
@@
 		(dnp no)
 		(fields_autoplaced yes)
-		(property "Reference" "#PWR093"
+		(property "Reference" "#PWR090"
 			(at 163.83 128.27 0)
 			(effects
@@
 		(on_board yes)
 		(dnp no)
-		(property "Reference" "R63"
+		(property "Reference" "R25"
 			(at 177.8 40.64 90)
 			(effects
@@
 		(dnp no)
 		(fields_autoplaced yes)
-		(property "Reference" "#PWR083"
+		(property "Reference" "#PWR080"
 			(at 104.14 69.85 0)
 			(effects
@@
 		(on_board yes)
 		(dnp no)
-		(property "Reference" "R69"
+		(property "Reference" "R31"
 			(at 71.12 74.9299 0)
 			(effects
@@
 		(on_board yes)
 		(dnp no)
-		(property "Reference" "C58"
+		(property "Reference" "C21"
 			(at 220.98 77.4699 0)
 			(effects
@@
 		(on_board yes)
 		(dnp no)
-		(property "Reference" "C59"
+		(property "Reference" "C22"
 			(at 232.41 77.4699 0)
 			(effects
@@
 		(dnp no)
 		(fields_autoplaced yes)
-		(property "Reference" "L4"
+		(property "Reference" "L1"
 			(at 193.04 31.75 90)
 			(effects
@@
 		(dnp no)
 		(fields_autoplaced yes)
-		(property "Reference" "#PWR089"
+		(property "Reference" "#PWR086"
 			(at 64.77 87.63 0)
 			(effects
@@
 		(dnp no)
 		(fields_autoplaced yes)
-		(property "Reference" "U14"
+		(property "Reference" "U11"
 			(at 77.47 39.37 0)
 			(effects
@@
 		(on_board yes)
 		(dnp no)
-		(property "Reference" "R65"
+		(property "Reference" "R27"
 			(at 175.26 53.3401 0)
 			(effects
@@
 		(dnp no)
 		(fields_autoplaced yes)
-		(property "Reference" "#PWR087"
+		(property "Reference" "#PWR084"
 			(at 251.46 71.12 0)
 			(effects
@@
 		(on_board yes)
 		(dnp no)
-		(property "Reference" "C64"
+		(property "Reference" "C27"
 			(at 46.99 138.4299 0)
 			(effects
@@
 		(on_board yes)
 		(dnp no)
-		(property "Reference" "C57"
+		(property "Reference" "C20"
 			(at 120.65 76.1999 0)
 			(effects
@@
 		(on_board yes)
 		(dnp no)
-		(property "Reference" "C65"
+		(property "Reference" "C28"
 			(at 95.25 143.5099 0)
 			(effects
@@
 		(on_board yes)
 		(dnp no)
-		(property "Reference" "C54"
+		(property "Reference" "C17"
 			(at 173.99 60.9599 0)
 			(effects
@@
 		(on_board yes)
 		(dnp no)
-		(property "Reference" "C63"
+		(property "Reference" "C26"
 			(at 83.82 125.476 90)
 			(effects
@@
 		(on_board yes)
 		(dnp no)
-		(property "Reference" "C68"
+		(property "Reference" "C31"
 			(at 124.46 144.272 90)
 			(effects
@@
 		(dnp no)
 		(fields_autoplaced yes)
-		(property "Reference" "L5"
+		(property "Reference" "L2"
 			(at 116.84 57.1499 0)
 			(effects
@@
 		(dnp no)
 		(fields_autoplaced yes)
-		(property "Reference" "U16"
+		(property "Reference" "U13"
 			(at 63.5 127 0)
 			(effects
@@
 		(on_board yes)
 		(dnp no)
-		(property "Reference" "R71"
+		(property "Reference" "R33"
 			(at 190.5 76.1999 0)
 			(effects
@@
 		(dnp no)
 		(fields_autoplaced yes)
-		(property "Reference" "#PWR086"
+		(property "Reference" "#PWR083"
 			(at 50.8 73.66 0)
 			(effects
@@
 		(on_board yes)
 		(dnp no)
-		(property "Reference" "R68"
+		(property "Reference" "R30"
 			(at 62.23 74.9299 0)
 			(effects
@@
 		(on_board yes)
 		(dnp no)
-		(property "Reference" "C67"
+		(property "Reference" "C30"
 			(at 119.38 144.272 90)
 			(effects
@@
 		(on_board yes)
 		(dnp no)
-		(property "Reference" "R70"
+		(property "Reference" "R32"
 			(at 181.61 76.1999 0)
 			(effects
@@
 		(on_board yes)
 		(dnp no)
-		(property "Reference" "C55"
+		(property "Reference" "C18"
 			(at 93.9863 81.28 90)
 			(effects
@@
 		(dnp yes)
 		(fields_autoplaced yes)
-		(property "Reference" "TP?"
+		(property "Reference" "TP9"
 			(at 91.44 128.7779 0)
 			(effects
@@
 		)
 		(instances
-			(project "SupercapManager"
-				(path "/6197145b-e7d4-44cc-9d90-537b6501bf60/2b4de7d2-e111-42d9-afee-f810f96a2f61"
-					(reference "TP?")
-					(unit 1)
-				)
-			)
 			(project "Rev 1B"
 				(path "/e5f99deb-ef42-4c5f-b80a-388477910e20/1e0b2151-e075-4f05-b22a-12d6722ef31a"
@@
 		(on_board yes)
 		(dnp no)
-		(property "Reference" "C53"
+		(property "Reference" "C16"
 			(at 54.61 59.6899 0)
 			(effects
@@
 		(on_board yes)
 		(dnp no)
-		(property "Reference" "C52"
+		(property "Reference" "C15"
 			(at 214.63 57.15 0)
 			(effects
@@
 		(dnp yes)
 		(fields_autoplaced yes)
-		(property "Reference" "TP2"
+		(property "Reference" "TP8"
 			(at 116.84 44.9579 0)
 			(effects
