File: Rev 1 Boards/Housekeeping Rev1/Housekeeping Rev1.kicad_pcb (KiCad board)
At the start: 2 copper layers, 0 parts

Commit message: beginning layout work for housekeeping pcb
Parts:
- added C1: 100u, Capacitor_THT:CP_Radial_D8.0mm_P3.50mm, F.Cu at (84.5, 130.5)
- added C10: 470p, Capacitor_SMD:C_0603_1608Metric_Pad1.08x0.95mm_HandSolder, F.Cu at (112.4, 52.0)
- added C11: 470u, Capacitor_THT:CP_Radial_D6.3mm_P2.50mm, F.Cu at (98.6, 35.2)
- added C12: 470u, Capacitor_THT:CP_Radial_D6.3mm_P2.50mm, F.Cu at (98.6, 43.1)
- added C2: 100u, Capacitor_THT:CP_Radial_D8.0mm_P3.50mm, F.Cu at (80.0, 29.9)
- added C3: 470p, Capacitor_SMD:C_0603_1608Metric_Pad1.08x0.95mm_HandSolder, F.Cu at (87.6, 149.5)
- added C4: 470p, Capacitor_SMD:C_0603_1608Metric_Pad1.08x0.95mm_HandSolder, F.Cu at (112.4, 47.0)
- added C5: 470u, Capacitor_THT:CP_Radial_D6.3mm_P2.50mm, F.Cu at (99.0, 158.0)
- added C6: 470u, Capacitor_THT:CP_Radial_D6.3mm_P2.50mm, F.Cu at (98.6, 27.4)
- added C7: 100u, Capacitor_THT:CP_Radial_D8.0mm_P3.50mm, F.Cu at (80.0, 39.5)
- added C8: 100u, Capacitor_THT:CP_Radial_D8.0mm_P3.50mm, F.Cu at (80.0, 49.0)
- added C9: 470p, Capacitor_SMD:C_0603_1608Metric_Pad1.08x0.95mm_HandSolder, F.Cu at (112.4, 49.5)
- added D1: BAT54, Package_TO_SOT_SMD:SOT-23_Handsoldering, F.Cu at (86.5, 168.5)
- added D2: BAT54, Package_TO_SOT_SMD:SOT-23_Handsoldering, F.Cu at (107.0, 50.5)
- added D3: BAT54, Package_TO_SOT_SMD:SOT-23_Handsoldering, F.Cu at (107.0, 55.3)
- added D4: BAT54, Package_TO_SOT_SMD:SOT-23_Handsoldering, F.Cu at (107.0, 60.0)
- added J1: Conn_01x02_Socket, Connector:Banana_Jack_2Pin, F.Cu at (34.4, 21.6)
- added J2: Conn_01x02_Socket, Connector:Banana_Jack_2Pin, F.Cu at (54.0, 157.0)
- added J3: Conn_01x02_Socket, Connector:Banana_Jack_2Pin, F.Cu at (63.0, 172.5)
- added J4: Conn_01x02_Socket, Connector:Banana_Jack_2Pin, F.Cu at (34.4, 57.8)
- added J5: Conn_01x02_Socket, Connector:Banana_Jack_2Pin, F.Cu at (34.4, 69.8)
- added J6: Conn_01x02_Socket, Connector:Banana_Jack_2Pin, F.Cu at (34.4, 81.9)
- added L1: 220u, ! Robomaster Passives:ASPIAIGS6055221MT, F.Cu at (87.5, 158.0)
- added L2: 220u, ! Robomaster Passives:ASPIAIGS6055221MT, F.Cu at (91.1, 29.3)
- added L3: 88u, ! Robomaster Passives:ASPIAIGS6055221MT, F.Cu at (91.1, 38.4)
- added L4: 220u, ! Robomaster Passives:ASPIAIGS6055221MT, F.Cu at (91.1, 47.5)
- added R1: 50, Resistor_SMD:R_0603_1608Metric_Pad0.98x0.95mm_HandSolder, F.Cu at (68.0, 184.5)
- added R10: 3.6k, Resistor_SMD:R_0603_1608Metric_Pad0.98x0.95mm_HandSolder, F.Cu at (116.7, 52.0)
- added R11: 0.33, Resistor_SMD:R_0603_1608Metric_Pad0.98x0.95mm_HandSolder, F.Cu at (116.7, 54.5)
- added R12: 0.24, Resistor_SMD:R_0603_1608Metric_Pad0.98x0.95mm_HandSolder, F.Cu at (116.7, 57.0)
- added R13: 2.2k, Resistor_SMD:R_0603_1608Metric_Pad0.98x0.95mm_HandSolder, F.Cu at (121.1, 44.5)
- added R14: 3.6k, Resistor_SMD:R_0603_1608Metric_Pad0.98x0.95mm_HandSolder, F.Cu at (121.1, 47.0)
- added R15: 3.6k, Resistor_SMD:R_0603_1608Metric_Pad0.98x0.95mm_HandSolder, F.Cu at (121.1, 49.5)
- added R16: 2.2k, Resistor_SMD:R_0603_1608Metric_Pad0.98x0.95mm_HandSolder, F.Cu at (121.1, 52.0)
- added R2: 50, Resistor_SMD:R_0603_1608Metric_Pad0.98x0.95mm_HandSolder, F.Cu at (72.6, 19.4)
- added R3: 50, Resistor_SMD:R_0603_1608Metric_Pad0.98x0.95mm_HandSolder, F.Cu at (72.6, 21.9)
- added R4: 50, Resistor_SMD:R_0603_1608Metric_Pad0.98x0.95mm_HandSolder, F.Cu at (72.6, 24.4)
- added R5: 0.33, Resistor_SMD:R_0603_1608Metric_Pad0.98x0.95mm_HandSolder, F.Cu at (71.6, 167.5)
- added R6: 0.33, Resistor_SMD:R_0603_1608Metric_Pad0.98x0.95mm_HandSolder, F.Cu at (112.4, 57.0)
- added R7: 2.2k, Resistor_SMD:R_0603_1608Metric_Pad0.98x0.95mm_HandSolder, F.Cu at (70.4, 149.5)
- added R8: 1.2k, Resistor_SMD:R_0603_1608Metric_Pad0.98x0.95mm_HandSolder, F.Cu at (116.7, 47.0)
- added R9: 3.6k, Resistor_SMD:R_0603_1608Metric_Pad0.98x0.95mm_HandSolder, F.Cu at (70.4, 142.5)
- added TP10: V_{E}, TestPoint:TestPoint_Bridge_Pitch2.0mm_Drill0.7mm, F.Cu at (85.0, 180.5)
- added TP11: V_{C}, TestPoint:TestPoint_Bridge_Pitch2.0mm_Drill0.7mm, F.Cu at (105.5, 31.1)
- added TP12: V_{E}, TestPoint:TestPoint_Bridge_Pitch2.0mm_Drill0.7mm, F.Cu at (105.5, 34.6)
- added TP13: V_{C}, TestPoint:TestPoint_Bridge_Pitch2.0mm_Drill0.7mm, F.Cu at (105.5, 38.0)
- added TP14: V_{E}, TestPoint:TestPoint_Bridge_Pitch2.0mm_Drill0.7mm, F.Cu at (105.5, 41.5)
- added TP7: V_{C}, TestPoint:TestPoint_Bridge_Pitch2.0mm_Drill0.7mm, F.Cu at (105.5, 17.3)
- added TP8: V_{E}, TestPoint:TestPoint_Bridge_Pitch2.0mm_Drill0.7mm, F.Cu at (105.5, 20.8)
- added TP9: V_{C}, TestPoint:TestPoint_Bridge_Pitch2.0mm_Drill0.7mm, F.Cu at (108.5, 151.5)
- added U1: MC34063A, Package_SO:SOIC-8_3.9x4.9mm_P1.27mm, F.Cu at (72.0, 157.5)
- added U2: MC34063A, Package_SO:SOIC-8_3.9x4.9mm_P1.27mm, F.Cu at (113.4, 25.6)
- added U3: MC34063A, Package_SO:SOIC-8_3.9x4.9mm_P1.27mm, F.Cu at (113.4, 32.1)
- added U4: MC34063A, Package_SO:SOIC-8_3.9x4.9mm_P1.27mm, F.Cu at (113.4, 38.7)
Routing:
- net Net-(D1-K): track 0.00 -> 33.4 mm
- net /+24_{MiniPC}: track 0.00 -> 15.9 mm
- net Net-(U1-CT): track 0.00 -> 15.5 mm
- net Net-(U1-COMP-): track 0.00 -> 13.1 mm
- net +3V3: track 0.00 -> 9.25 mm
- net Net-(U1-DC): track 0.00 -> 6.22 mm
