File: Rev 1B Boards/Rev 1B/Rev 1B.kicad_pcb (KiCad board)
At the start: 2 copper layers, 0 parts

Commit message: Begin layout
Completed ideal diode layout
Parts:
- added C1: 0.1u, Capacitor_SMD:C_0603_1608Metric_Pad1.08x0.95mm_HandSolder, F.Cu at (370.2, 85.6)
- added C10: 0.1u, Capacitor_SMD:C_0603_1608Metric_Pad1.08x0.95mm_HandSolder, F.Cu at (202.9, 59.6)
- added C11: 0.1u, Capacitor_SMD:C_0603_1608Metric_Pad1.08x0.95mm_HandSolder, F.Cu at (202.9, 62.1)
- added C12: 0.1u, Capacitor_SMD:C_0603_1608Metric_Pad1.08x0.95mm_HandSolder, F.Cu at (207.3, 52.1)
- added C13: 6.8u, Capacitor_SMD:C_0603_1608Metric_Pad1.08x0.95mm_HandSolder, F.Cu at (207.3, 54.6)
- added C14: 82p, Capacitor_SMD:C_0603_1608Metric_Pad1.08x0.95mm_HandSolder, F.Cu at (94.0, 28.0)
- added C15: 100p, Capacitor_SMD:C_0603_1608Metric_Pad1.08x0.95mm_HandSolder, F.Cu at (94.0, 30.5)
- added C16: 1u, Capacitor_SMD:C_0603_1608Metric_Pad1.08x0.95mm_HandSolder, F.Cu at (94.0, 33.0)
- added C17: 1u, Capacitor_SMD:C_0603_1608Metric_Pad1.08x0.95mm_HandSolder, F.Cu at (94.0, 35.5)
- added C18: 0.01u, Capacitor_SMD:C_0603_1608Metric_Pad1.08x0.95mm_HandSolder, F.Cu at (94.0, 38.0)
- added C19: 0.01u, Capacitor_SMD:C_0603_1608Metric_Pad1.08x0.95mm_HandSolder, F.Cu at (94.0, 40.5)
- added C2: 0.1u, Capacitor_SMD:C_0603_1608Metric_Pad1.08x0.95mm_HandSolder, F.Cu at (370.2, 88.1)
- added C20: 10u, Capacitor_SMD:C_1206_3216Metric_Pad1.33x1.80mm_HandSolder, F.Cu at (82.8, 28.4)
- added C21: 10u, Capacitor_SMD:C_1206_3216Metric_Pad1.33x1.80mm_HandSolder, F.Cu at (82.8, 31.8)
- added C22: 10u, Capacitor_SMD:C_1206_3216Metric_Pad1.33x1.80mm_HandSolder, F.Cu at (82.8, 35.1)
- added C23: 10u, Capacitor_SMD:C_1206_3216Metric_Pad1.33x1.80mm_HandSolder, F.Cu at (82.8, 38.5)
- added C24: 10u, Capacitor_SMD:C_1206_3216Metric_Pad1.33x1.80mm_HandSolder, F.Cu at (82.8, 41.8)
- added C25: 100u, Capacitor_THT:CP_Radial_D8.0mm_P3.50mm, F.Cu at (104.3, 61.0)
- added C26: 0.1u, Capacitor_SMD:C_0603_1608Metric_Pad1.08x0.95mm_HandSolder, F.Cu at (94.0, 43.0)
- added C27: 10u, Capacitor_SMD:C_1206_3216Metric_Pad1.33x1.80mm_HandSolder, F.Cu at (82.8, 45.1)
- added C28: 330p, Capacitor_SMD:C_0603_1608Metric_Pad1.08x0.95mm_HandSolder, F.Cu at (98.3, 28.0)
- added C29: 10u, Capacitor_SMD:C_1206_3216Metric_Pad1.33x1.80mm_HandSolder, F.Cu at (88.8, 28.4)
- added C3: 0.1u, Capacitor_SMD:C_0603_1608Metric_Pad1.08x0.95mm_HandSolder, F.Cu at (370.2, 90.6)
- added C30: 10u, Capacitor_SMD:C_1206_3216Metric_Pad1.33x1.80mm_HandSolder, F.Cu at (88.8, 31.8)
- added C31: 10u, Capacitor_SMD:C_1206_3216Metric_Pad1.33x1.80mm_HandSolder, F.Cu at (88.8, 35.1)
- added C32: 10u, Capacitor_SMD:C_1206_3216Metric_Pad1.33x1.80mm_HandSolder, F.Cu at (88.8, 38.5)
- added C33: 10u, Capacitor_SMD:C_1206_3216Metric_Pad1.33x1.80mm_HandSolder, F.Cu at (88.8, 41.8)
- added C34: 0.022u, Capacitor_SMD:C_0603_1608Metric_Pad1.08x0.95mm_HandSolder, F.Cu at (210.5, 170.7)
- added C35: 47u, Capacitor_SMD:C_1206_3216Metric_Pad1.33x1.80mm_HandSolder, F.Cu at (222.5, 170.9)
- added C36: 0.1u, Capacitor_SMD:C_0603_1608Metric_Pad1.08x0.95mm_HandSolder, F.Cu at (213.9, 173.7)
- added C37: 10u, Capacitor_SMD:C_1206_3216Metric_Pad1.33x1.80mm_HandSolder, F.Cu at (258.1, 249.3)
- added C38: 10u, Capacitor_SMD:C_1206_3216Metric_Pad1.33x1.80mm_HandSolder, F.Cu at (258.1, 252.7)
- added C39: 2.2u, Capacitor_THT:C_Radial_D5.0mm_H11.0mm_P2.00mm, F.Cu at (263.4, 260.5)
- added C4: 1000p, Capacitor_SMD:C_0603_1608Metric_Pad1.08x0.95mm_HandSolder, F.Cu at (370.2, 93.1)
- added C40: 1u, Capacitor_SMD:C_0603_1608Metric_Pad1.08x0.95mm_HandSolder, F.Cu at (238.7, 248.9)
- added C41: 10u, Capacitor_SMD:C_1206_3216Metric_Pad1.33x1.80mm_HandSolder, F.Cu at (258.1, 256.0)
- added C42: 10u, Capacitor_SMD:C_1206_3216Metric_Pad1.33x1.80mm_HandSolder, F.Cu at (258.1, 259.4)
- added C43: 10u, Capacitor_SMD:C_1206_3216Metric_Pad1.33x1.80mm_HandSolder, F.Cu at (258.1, 262.7)
- added C44: 15p, Capacitor_SMD:C_0603_1608Metric_Pad1.08x0.95mm_HandSolder, F.Cu at (238.7, 251.4)
- added C45: 0.1u, Capacitor_SMD:C_0603_1608Metric_Pad1.08x0.95mm_HandSolder, F.Cu at (238.7, 253.9)
- added C46: 0.1u, Capacitor_SMD:C_0603_1608Metric_Pad1.08x0.95mm_HandSolder, F.Cu at (238.7, 256.4)
- added C47: 1u, Capacitor_SMD:C_0603_1608Metric_Pad1.08x0.95mm_HandSolder, F.Cu at (238.7, 258.9)
- added C48: 1u, Capacitor_SMD:C_0603_1608Metric_Pad1.08x0.95mm_HandSolder, F.Cu at (238.7, 261.5)
- added C49: 0.1u, Capacitor_SMD:C_0603_1608Metric_Pad1.08x0.95mm_HandSolder, F.Cu at (238.7, 264.0)
- added C5: 0.1u, Capacitor_SMD:C_0603_1608Metric_Pad1.08x0.95mm_HandSolder, F.Cu at (370.2, 95.6)
- added C50: 0.1u, Capacitor_SMD:C_0603_1608Metric_Pad1.08x0.95mm_HandSolder, F.Cu at (110.7, 242.3)
- added C51: 220u, Capacitor_THT:CP_Radial_D6.3mm_P2.50mm, F.Cu at (94.6, 227.7)
- added C52: 220u, Capacitor_THT:CP_Radial_D6.3mm_P2.50mm, F.Cu at (94.6, 235.6)
- added C53: 220u, Capacitor_THT:CP_Radial_D6.3mm_P2.50mm, F.Cu at (94.6, 243.4)
- added C54: 220u, Capacitor_THT:CP_Radial_D6.3mm_P2.50mm, F.Cu at (94.6, 251.2)
- added C55: 220u, Capacitor_THT:CP_Radial_D6.3mm_P2.50mm, F.Cu at (94.6, 259.1)
- added C56: 0.1u, Capacitor_SMD:C_0603_1608Metric_Pad1.08x0.95mm_HandSolder, F.Cu at (110.7, 244.8)
- added C57: 200p, Capacitor_SMD:C_0603_1608Metric_Pad1.08x0.95mm_HandSolder, F.Cu at (110.7, 247.3)
- added C58: 0.47u, Capacitor_SMD:C_0603_1608Metric_Pad1.08x0.95mm_HandSolder, F.Cu at (110.7, 249.8)
- added C59: 4.7u, Capacitor_SMD:C_0603_1608Metric_Pad1.08x0.95mm_HandSolder, F.Cu at (110.7, 252.3)
- added C6: 1000p, Capacitor_SMD:C_0603_1608Metric_Pad1.08x0.95mm_HandSolder, F.Cu at (370.2, 98.1)
- added C60: 0.47u, Capacitor_SMD:C_0603_1608Metric_Pad1.08x0.95mm_HandSolder, F.Cu at (115.0, 242.3)
- added C61: 0.015u, Capacitor_SMD:C_0603_1608Metric_Pad1.08x0.95mm_HandSolder, F.Cu at (115.0, 244.8)
- added C62: 220u, Capacitor_THT:CP_Radial_D6.3mm_P2.50mm, F.Cu at (88.9, 125.6)
- added C63: 0.1u, Capacitor_SMD:C_0603_1608Metric_Pad1.08x0.95mm_HandSolder, F.Cu at (96.3, 136.9)
- added C64: 0.1u, Capacitor_SMD:C_0603_1608Metric_Pad1.08x0.95mm_HandSolder, F.Cu at (96.3, 139.5)
- added C65: 220u, Capacitor_THT:CP_Radial_D6.3mm_P2.50mm, F.Cu at (88.9, 133.4)
- added C66: 220u, Capacitor_THT:CP_Radial_D6.3mm_P2.50mm, F.Cu at (88.9, 141.3)
- added C67: 1u, Capacitor_SMD:C_0603_1608Metric_Pad1.08x0.95mm_HandSolder, F.Cu at (96.3, 142.0)
- added C68: 1u, Capacitor_SMD:C_0603_1608Metric_Pad1.08x0.95mm_HandSolder, F.Cu at (96.3, 144.5)
- added C69: 10u, Capacitor_SMD:C_1206_3216Metric_Pad1.33x1.80mm_HandSolder, F.Cu at (115.6, 142.7)
- added C7: 0.1u, Capacitor_SMD:C_0603_1608Metric_Pad1.08x0.95mm_HandSolder, F.Cu at (202.9, 52.1)
- added C70: 15p, Capacitor_SMD:C_0603_1608Metric_Pad1.08x0.95mm_HandSolder, F.Cu at (96.3, 147.0)
- added C71: 180p, Capacitor_SMD:C_0603_1608Metric_Pad1.08x0.95mm_HandSolder, F.Cu at (96.3, 149.5)
- added C72: 0.1u, Capacitor_SMD:C_0603_1608Metric_Pad1.08x0.95mm_HandSolder, F.Cu at (100.6, 136.9)
- added C73: 0.01u, Capacitor_SMD:C_0603_1608Metric_Pad1.08x0.95mm_HandSolder, F.Cu at (100.6, 139.5)
- added C74: 110, Capacitor_THT:C_Radial_D18.0mm_H35.5mm_P7.50mm, F.Cu at (368.3, 165.1)
- added C75: 110, Capacitor_THT:C_Radial_D18.0mm_H35.5mm_P7.50mm, F.Cu at (368.3, 184.7)
- added C76: 110, Capacitor_THT:C_Radial_D18.0mm_H35.5mm_P7.50mm, F.Cu at (368.3, 204.2)
- added C77: 110, Capacitor_THT:C_Radial_D18.0mm_H35.5mm_P7.50mm, F.Cu at (368.3, 223.8)
- added C78: 100p, Capacitor_SMD:C_0603_1608Metric_Pad1.08x0.95mm_HandSolder, F.Cu at (356.6, 185.9)
- added C79: 0.1u, Capacitor_SMD:C_0603_1608Metric_Pad1.08x0.95mm_HandSolder, F.Cu at (356.6, 188.4)
- added C8: 0.1u, Capacitor_SMD:C_0603_1608Metric_Pad1.08x0.95mm_HandSolder, F.Cu at (202.9, 54.6)
- added C9: 0.1u, Capacitor_SMD:C_0603_1608Metric_Pad1.08x0.95mm_HandSolder, F.Cu at (202.9, 57.1)
- added D1: MMSZ4678T1G, Diode_SMD:D_SOD-123, F.Cu at (371.0, 106.1)
- added D2: BAT54, Package_TO_SOT_SMD:SOT-23_Handsoldering, F.Cu at (88.4, 49.3)
- added D3: BAT54, Package_TO_SOT_SMD:SOT-23_Handsoldering, F.Cu at (88.4, 54.1)
- added D4: BAT54, Package_TO_SOT_SMD:SOT-23_Handsoldering, F.Cu at (264.3, 250.2)
- added D5: BAT54, Package_TO_SOT_SMD:SOT-23_Handsoldering, F.Cu at (264.3, 254.9)
- added D6: LTST-C193TBKT-5A, LED_SMD:LED_0603_1608Metric_Pad1.05x0.95mm_HandSolder, F.Cu at (242.8, 272.3)
- added D7: LTST-C193KSKT-5A, LED_SMD:LED_0603_1608Metric_Pad1.05x0.95mm_HandSolder, F.Cu at (242.8, 274.9)
- added J1: Conn_01x01_Pin, Connector_Wire:SolderWire-2.5sqmm_1x01_D2.4mm_OD3.6mm, F.Cu at (357.4, 31.6)
- added J10: Conn_01x01_Pin, Connector_Wire:SolderWire-2.5sqmm_1x01_D2.4mm_OD3.6mm, F.Cu at (363.5, 37.7)
- added J11: Banana 2P, Connector:Banana_Jack_2Pin, F.Cu at (197.7, 91.0)
- added J12: Banana 2P, Connector:Banana_Jack_2Pin, F.Cu at (197.7, 103.1)
- added J13: Banana 2P, Connector:Banana_Jack_2Pin, F.Cu at (318.2, 71.8)
- added J14: Banana 2P, Connector:Banana_Jack_2Pin, F.Cu at (318.2, 83.8)
- added J15: Banana 2P, Connector:Banana_Jack_2Pin, F.Cu at (29.4, 75.8)
- added J16: Banana 2P, Connector:Banana_Jack_2Pin, F.Cu at (193.4, 253.3)
- added J17: Banana 2P, Connector:Banana_Jack_2Pin, F.Cu at (193.4, 265.4)
- added J18: Banana 2P, Connector:Banana_Jack_2Pin, F.Cu at (50.1, 231.0)
- added J19: Banana 2P, Connector:Banana_Jack_2Pin, F.Cu at (50.1, 243.1)
- added J2: Conn_01x01_Pin, Connector_Wire:SolderWire-2.5sqmm_1x01_D2.4mm_OD3.6mm, F.Cu at (357.4, 37.7)
- added J20: Banana 2P, Connector:Banana_Jack_2Pin, F.Cu at (50.1, 255.1)
- added J21: Banana 2P, Connector:Banana_Jack_2Pin, F.Cu at (27.6, 32.5)
- added J22: Banana 2P, Connector:Banana_Jack_2Pin, F.Cu at (27.6, 44.6)
- added J23: Conn_01x01_Pin, Connector_Wire:SolderWire-2.5sqmm_1x01_D2.4mm_OD3.6mm, F.Cu at (240.8, 235.6)
- added J24: Banana 2P, Connector:Banana_Jack_2Pin, F.Cu at (27.6, 56.6)
- added J25: Banana 2P, Connector:Banana_Jack_2Pin, F.Cu at (200.3, 155.9)
- added J26: Banana 2P, Connector:Banana_Jack_2Pin, F.Cu at (233.1, 156.3)
- added J27: Banana 2P, Connector:Banana_Jack_2Pin, F.Cu at (45.0, 131.0)
- added J28: Banana 2P, Connector:Banana_Jack_2Pin, F.Cu at (45.0, 143.1)
- added J29: Conn_01x02_Socket, Connector_PinSocket_2.00mm:PinSocket_1x02_P2.00mm_Vertical, F.Cu at (238.6, 267.2)
- added J3: Conn_01x01_Pin, Connector_Wire:SolderWire-2.5sqmm_1x01_D2.4mm_OD3.6mm, F.Cu at (236.8, 64.0)
- added J30: XT30_F, Connector_AMASS:AMASS_XT30U-F_1x02_P5.0mm_Vertical, F.Cu at (333.6, 188.2)
- added J31: XT30_F, Connector_AMASS:AMASS_XT30U-F_1x02_P5.0mm_Vertical, F.Cu at (333.6, 195.5)
- added J4: Banana 2P, Connector:Banana_Jack_2Pin, F.Cu at (318.3, 34.6)
- added J5: Banana 2P, Connector:Banana_Jack_2Pin, F.Cu at (318.3, 46.7)
- added J6: JST4_F, Connector_JST:JST_GH_BM04B-GHS-TBT_1x04-1MP_P1.25mm_Vertical, F.Cu at (238.9, 90.2)
- added J7: Conn_01x01_Pin, Connector_Wire:SolderWire-2.5sqmm_1x01_D2.4mm_OD3.6mm, F.Cu at (236.8, 70.0)
- added J8: Banana 2P, Connector:Banana_Jack_2Pin, F.Cu at (318.3, 58.7)
- added J9: Conn_01x01_Pin, Connector_Wire:SolderWire-2.5sqmm_1x01_D2.4mm_OD3.6mm, F.Cu at (242.9, 51.9)
- added L1: 220u, ! Robomaster Passives:ASPIAIGS6055221MT, F.Cu at (96.4, 48.8)
- added L2: 220u, ! Robomaster Passives:ASPIAIGS6055221MT, F.Cu at (96.4, 57.9)
- added L3: 8.2u, Inductor_SMD:L_10.4x10.4_H4.8, F.Cu at (107.4, 50.3)
- added L4: 4.7u, Inductor_SMD:L_Bourns_SRN8040TA, F.Cu at (263.4, 269.7)
- added L5: 1.8u, Inductor_SMD:L_Bourns_SRP1245A, F.Cu at (113.1, 230.8)
- added L6: 1.8u, Inductor_SMD:L_Bourns_SRP1245A, F.Cu at (102.0, 128.7)
- added Q1: BSC059N04LS6, Package_SON:Infineon_PG-TDSON-8_6.15x5.15mm, F.Cu at (358.9, 56.1)
- added Q10: 2SCR587D3, Package_TO_SOT_SMD:TO-252-2, F.Cu at (349.1, 188.8)
- added Q11: 2SAR587D3, Package_TO_SOT_SMD:TO-252-2, F.Cu at (349.1, 197.0)
- added Q2: BSC059N04LS6, Package_SON:Infineon_PG-TDSON-8_6.15x5.15mm, F.Cu at (358.9, 62.8)
- added Q3: BSC059N04LS6, Package_SON:Infineon_PG-TDSON-8_6.15x5.15mm, F.Cu at (216.0, 166.9)
- added Q4: BSC059N04LS6, Package_SON:Infineon_PG-TDSON-8_6.15x5.15mm, F.Cu at (254.2, 268.2)
- added Q5: BSC059N04LS6, Package_SON:Infineon_PG-TDSON-8_6.15x5.15mm, F.Cu at (254.2, 274.9)
- added Q6: BSC059N04LS6, Package_SON:Infineon_PG-TDSON-8_6.15x5.15mm, F.Cu at (104.3, 244.4)
- added Q7: BSC059N04LS6, Package_SON:Infineon_PG-TDSON-8_6.15x5.15mm, F.Cu at (104.3, 251.1)
- added Q8: BSC059N04LS6, Package_SON:Infineon_PG-TDSON-8_6.15x5.15mm, F.Cu at (114.4, 125.0)
- added Q9: BSC059N04LS6, Package_SON:Infineon_PG-TDSON-8_6.15x5.15mm, F.Cu at (114.4, 131.7)
- added R1: 0, Resistor_SMD:R_0603_1608Metric_Pad0.98x0.95mm_HandSolder, F.Cu at (356.5, 75.1)
- added R10: 100k, Resistor_SMD:R_0603_1608Metric_Pad0.98x0.95mm_HandSolder, F.Cu at (374.6, 95.6)
- added R11: 1Meg, Resistor_SMD:R_0603_1608Metric_Pad0.98x0.95mm_HandSolder, F.Cu at (374.6, 98.1)
- added R12: 1Meg, Resistor_SMD:R_0603_1608Metric_Pad0.98x0.95mm_HandSolder, F.Cu at (374.6, 100.6)
- added R13: 1k, Resistor_SMD:R_0603_1608Metric_Pad0.98x0.95mm_HandSolder, F.Cu at (374.6, 103.1)
- added R14: 100k, Resistor_SMD:R_0603_1608Metric_Pad0.98x0.95mm_HandSolder, F.Cu at (378.9, 85.6)
- added R15: 1Meg, Resistor_SMD:R_0603_1608Metric_Pad0.98x0.95mm_HandSolder, F.Cu at (378.9, 88.1)
- added R16: 15k, Resistor_SMD:R_0603_1608Metric_Pad0.98x0.95mm_HandSolder, F.Cu at (378.9, 90.6)
- added R17: 47k, Resistor_SMD:R_0603_1608Metric_Pad0.98x0.95mm_HandSolder, F.Cu at (378.9, 93.1)
- added R18: 1Meg, Resistor_SMD:R_0603_1608Metric_Pad0.98x0.95mm_HandSolder, F.Cu at (378.9, 95.6)
- added R19: 1.5k, Resistor_SMD:R_0603_1608Metric_Pad0.98x0.95mm_HandSolder, F.Cu at (207.3, 57.1)
- added R2: 0, Resistor_SMD:R_0603_1608Metric_Pad0.98x0.95mm_HandSolder, F.Cu at (356.5, 77.6)
- added R20: 1.5k, Resistor_SMD:R_0603_1608Metric_Pad0.98x0.95mm_HandSolder, F.Cu at (207.3, 59.6)
- added R21: 1.5k, Resistor_SMD:R_0603_1608Metric_Pad0.98x0.95mm_HandSolder, F.Cu at (207.3, 62.1)
- added R22: 1.5k, Resistor_SMD:R_0603_1608Metric_Pad0.98x0.95mm_HandSolder, F.Cu at (211.6, 52.1)
- added R23: 180k, Resistor_SMD:R_0603_1608Metric_Pad0.98x0.95mm_HandSolder, F.Cu at (211.6, 54.6)
- added R24: 220k, Resistor_SMD:R_0603_1608Metric_Pad0.98x0.95mm_HandSolder, F.Cu at (211.6, 57.1)
- added R25: 180, Resistor_SMD:R_0805_2012Metric_Pad1.20x1.40mm_HandSolder, F.Cu at (87.6, 62.6)
- added R26: 1, Resistor_SMD:R_0603_1608Metric_Pad0.98x0.95mm_HandSolder, F.Cu at (98.3, 30.5)
- added R27: 1, Resistor_SMD:R_0603_1608Metric_Pad0.98x0.95mm_HandSolder, F.Cu at (98.3, 33.0)
- added R28: 1.2k, Resistor_SMD:R_0603_1608Metric_Pad0.98x0.95mm_HandSolder, F.Cu at (98.3, 35.5)
- added R29: 22k, Resistor_SMD:R_0603_1608Metric_Pad0.98x0.95mm_HandSolder, F.Cu at (98.3, 38.0)
- added R3: 0.02, Resistor_SMD:R_0805_2012Metric_Pad1.20x1.40mm_HandSolder, F.Cu at (376.2, 105.9)
- added R30: 180k, Resistor_SMD:R_0603_1608Metric_Pad0.98x0.95mm_HandSolder, F.Cu at (98.3, 40.5)
- added R31: 820, Resistor_SMD:R_0603_1608Metric_Pad0.98x0.95mm_HandSolder, F.Cu at (98.3, 43.0)
- added R32: 1k, Resistor_SMD:R_0603_1608Metric_Pad0.98x0.95mm_HandSolder, F.Cu at (102.7, 28.0)
- added R33: 22k, Resistor_SMD:R_0603_1608Metric_Pad0.98x0.95mm_HandSolder, F.Cu at (102.7, 30.5)
- added R34: 100k, Resistor_SMD:R_0603_1608Metric_Pad0.98x0.95mm_HandSolder, F.Cu at (102.7, 33.0)
- added R35: 13.7k, Resistor_SMD:R_0603_1608Metric_Pad0.98x0.95mm_HandSolder, F.Cu at (102.7, 35.5)
- added R36: 6.8, Resistor_SMD:R_0805_2012Metric_Pad1.20x1.40mm_HandSolder, F.Cu at (260.8, 275.9)
- added R37: 0, Resistor_SMD:R_0603_1608Metric_Pad0.98x0.95mm_HandSolder, F.Cu at (243.1, 248.9)
- added R38: 0.01, Resistor_SMD:R_0612_1632Metric_Pad1.18x3.40mm_HandSolder, F.Cu at (247.2, 273.5)
- added R39: 27k, Resistor_SMD:R_0603_1608Metric_Pad0.98x0.95mm_HandSolder, F.Cu at (243.1, 251.4)
- added R4: 1k, Resistor_SMD:R_0603_1608Metric_Pad0.98x0.95mm_HandSolder, F.Cu at (370.2, 100.6)
- added R40: 0, Resistor_SMD:R_0603_1608Metric_Pad0.98x0.95mm_HandSolder, F.Cu at (243.1, 253.9)
- added R41: 470k, Resistor_SMD:R_0603_1608Metric_Pad0.98x0.95mm_HandSolder, F.Cu at (243.1, 256.4)
- added R42: 15k, Resistor_SMD:R_0603_1608Metric_Pad0.98x0.95mm_HandSolder, F.Cu at (243.1, 258.9)
- added R43: 4.7k, Resistor_SMD:R_0603_1608Metric_Pad0.98x0.95mm_HandSolder, F.Cu at (243.1, 261.5)
- added R44: 4.7k, Resistor_SMD:R_0603_1608Metric_Pad0.98x0.95mm_HandSolder, F.Cu at (243.1, 264.0)
- added R45: 9.31k, Resistor_SMD:R_0603_1608Metric_Pad0.98x0.95mm_HandSolder, F.Cu at (247.4, 248.9)
- added R46: 82k, Resistor_SMD:R_0603_1608Metric_Pad0.98x0.95mm_HandSolder, F.Cu at (247.4, 251.4)
- added R47: 430k, Resistor_SMD:R_0603_1608Metric_Pad0.98x0.95mm_HandSolder, F.Cu at (247.4, 253.9)
- added R48: 47k, Resistor_SMD:R_0603_1608Metric_Pad0.98x0.95mm_HandSolder, F.Cu at (247.4, 256.4)
- added R49: 0, Resistor_SMD:R_0603_1608Metric_Pad0.98x0.95mm_HandSolder, F.Cu at (115.0, 247.3)
- added R5: 1Meg, Resistor_SMD:R_0603_1608Metric_Pad0.98x0.95mm_HandSolder, F.Cu at (370.2, 103.1)
- added R50: 2m, Resistor_SMD:R_2512_6332Metric_Pad1.40x3.35mm_HandSolder, F.Cu at (113.0, 256.0)
- added R51: 0, Resistor_SMD:R_0603_1608Metric_Pad0.98x0.95mm_HandSolder, F.Cu at (115.0, 249.8)
- added R52: 18k, Resistor_SMD:R_0603_1608Metric_Pad0.98x0.95mm_HandSolder, F.Cu at (115.0, 252.3)
- added R53: 35.7k, Resistor_SMD:R_0603_1608Metric_Pad0.98x0.95mm_HandSolder, F.Cu at (119.4, 242.3)
- added R54: 75k, Resistor_SMD:R_0603_1608Metric_Pad0.98x0.95mm_HandSolder, F.Cu at (119.4, 244.8)
- added R55: 39k, Resistor_SMD:R_0603_1608Metric_Pad0.98x0.95mm_HandSolder, F.Cu at (119.4, 247.3)
- added R56: 22k, Resistor_SMD:R_0603_1608Metric_Pad0.98x0.95mm_HandSolder, F.Cu at (119.4, 249.8)
- added R57: 470k, Resistor_SMD:R_0603_1608Metric_Pad0.98x0.95mm_HandSolder, F.Cu at (119.4, 252.3)
- added R58: 47m, Resistor_SMD:R_1206_3216Metric_Pad1.30x1.75mm_HandSolder, F.Cu at (115.6, 146.0)
- added R59: 1m, Resistor_SMD:R_0612_1632Metric_Pad1.18x3.40mm_HandSolder, F.Cu at (96.3, 153.2)
- added R6: 1k, Resistor_SMD:R_0603_1608Metric_Pad0.98x0.95mm_HandSolder, F.Cu at (374.6, 85.6)
- added R60: 1m, Resistor_SMD:R_0612_1632Metric_Pad1.18x3.40mm_HandSolder, F.Cu at (100.7, 153.2)
- added R61: 100k, Resistor_SMD:R_0603_1608Metric_Pad0.98x0.95mm_HandSolder, F.Cu at (100.6, 142.0)
- added R62: 0, Resistor_SMD:R_0603_1608Metric_Pad0.98x0.95mm_HandSolder, F.Cu at (100.6, 144.5)
- added R63: 0, Resistor_SMD:R_0603_1608Metric_Pad0.98x0.95mm_HandSolder, F.Cu at (100.6, 147.0)
- added R64: 22.6k, Resistor_SMD:R_0603_1608Metric_Pad0.98x0.95mm_HandSolder, F.Cu at (100.6, 149.5)
- added R65: 330k, Resistor_SMD:R_0603_1608Metric_Pad0.98x0.95mm_HandSolder, F.Cu at (105.0, 136.9)
- added R66: 0, Resistor_SMD:R_0603_1608Metric_Pad0.98x0.95mm_HandSolder, F.Cu at (105.0, 139.5)
- added R67: 76.8k, Resistor_SMD:R_0603_1608Metric_Pad0.98x0.95mm_HandSolder, F.Cu at (105.0, 142.0)
- added R68: 30k, Resistor_SMD:R_0603_1608Metric_Pad0.98x0.95mm_HandSolder, F.Cu at (105.0, 144.5)
- added R69: 43k, Resistor_SMD:R_0603_1608Metric_Pad0.98x0.95mm_HandSolder, F.Cu at (105.0, 147.0)
- added R7: 1Meg, Resistor_SMD:R_0603_1608Metric_Pad0.98x0.95mm_HandSolder, F.Cu at (374.6, 88.1)
- added R70: 1Meg, Resistor_SMD:R_0603_1608Metric_Pad0.98x0.95mm_HandSolder, F.Cu at (356.6, 190.9)
- added R71: 0.1, Resistor_SMD:R_1206_3216Metric_Pad1.30x1.75mm_HandSolder, F.Cu at (345.2, 202.7)
- added R72: 100, Resistor_SMD:R_0603_1608Metric_Pad0.98x0.95mm_HandSolder, F.Cu at (356.6, 193.4)
- added R73: 100, Resistor_SMD:R_0603_1608Metric_Pad0.98x0.95mm_HandSolder, F.Cu at (356.6, 195.9)
- added R74: 1Meg, Resistor_SMD:R_0603_1608Metric_Pad0.98x0.95mm_HandSolder, F.Cu at (356.6, 198.4)
- added R75: 0.1, Resistor_SMD:R_1206_3216Metric_Pad1.30x1.75mm_HandSolder, F.Cu at (345.2, 205.9)
- added R8: 47k, Resistor_SMD:R_0603_1608Metric_Pad0.98x0.95mm_HandSolder, F.Cu at (374.6, 90.6)
- added R9: 1k, Resistor_SMD:R_0603_1608Metric_Pad0.98x0.95mm_HandSolder, F.Cu at (374.6, 93.1)
- added TP1: V_{DIFF10}, TestPoint:TestPoint_Bridge_Pitch2.0mm_Drill0.7mm, F.Cu at (388.6, 104.0)
- added TP10: V_{HIDRV}, TestPoint:TestPoint_Bridge_Pitch2.0mm_Drill0.7mm, F.Cu at (251.3, 249.4)
- added TP11: V_{SW}, TestPoint:TestPoint_Bridge_Pitch2.0mm_Drill0.7mm, F.Cu at (251.3, 252.8)
- added TP12: V_{P}, TestPoint:TestPoint_Bridge_Pitch2.0mm_Drill0.7mm, F.Cu at (251.3, 256.3)
- added TP13: V_{LODRV}, TestPoint:TestPoint_Bridge_Pitch2.0mm_Drill0.7mm, F.Cu at (251.3, 259.7)
- added TP14: V_{N}, TestPoint:TestPoint_Bridge_Pitch2.0mm_Drill0.7mm, F.Cu at (251.3, 263.2)
- added TP15: V_{HO}, TestPoint:TestPoint_Bridge_Pitch2.0mm_Drill0.7mm, F.Cu at (101.5, 225.5)
- added TP16: V_{SW}, TestPoint:TestPoint_Bridge_Pitch2.0mm_Drill0.7mm, F.Cu at (101.5, 228.9)
- added TP17: V_{P}, TestPoint:TestPoint_Bridge_Pitch2.0mm_Drill0.7mm, F.Cu at (101.5, 232.4)
- added TP18: V_{LO}, TestPoint:TestPoint_Bridge_Pitch2.0mm_Drill0.7mm, F.Cu at (101.5, 235.8)
- added TP19: V_{N}, TestPoint:TestPoint_Bridge_Pitch2.0mm_Drill0.7mm, F.Cu at (101.5, 239.3)
- added TP2: V_{SCL}, TestPoint:TestPoint_Bridge_Pitch2.0mm_Drill0.7mm, F.Cu at (202.5, 65.1)
- added TP20: V_{SW}, TestPoint:TestPoint_Bridge_Pitch2.0mm_Drill0.7mm, F.Cu at (108.9, 137.4)
- added TP21: V_{P}, TestPoint:TestPoint_Bridge_Pitch2.0mm_Drill0.7mm, F.Cu at (108.9, 140.9)
- added TP22: V_{N}, TestPoint:TestPoint_Bridge_Pitch2.0mm_Drill0.7mm, F.Cu at (108.9, 144.3)
- added TP23: V_{LDRV}, TestPoint:TestPoint_Bridge_Pitch2.0mm_Drill0.7mm, F.Cu at (108.9, 147.8)
- added TP24: V_{HDRV}, TestPoint:TestPoint_Bridge_Pitch2.0mm_Drill0.7mm, F.Cu at (108.9, 151.2)
- added TP25: V_{OUT}, TestPoint:TestPoint_Bridge_Pitch2.0mm_Drill0.7mm, F.Cu at (331.7, 200.8)
- added TP26: V_{CAP}, TestPoint:TestPoint_Bridge_Pitch2.0mm_Drill0.7mm, F.Cu at (331.7, 204.3)
- added TP27: V_{MID}, TestPoint:TestPoint_Bridge_Pitch2.0mm_Drill0.7mm, F.Cu at (331.7, 207.8)
- added TP28: V_{REF}, TestPoint:TestPoint_Bridge_Pitch2.0mm_Drill0.7mm, F.Cu at (331.7, 211.2)
- added TP3: V_{SDA}, TestPoint:TestPoint_Bridge_Pitch2.0mm_Drill0.7mm, F.Cu at (202.5, 68.5)
- added TP4: V_{SC+BUF}, TestPoint:TestPoint_Bridge_Pitch2.0mm_Drill0.7mm, F.Cu at (202.5, 72.0)
- added TP5: V_{C}, TestPoint:TestPoint_Bridge_Pitch2.0mm_Drill0.7mm, F.Cu at (81.5, 48.5)
- added TP6: V_{C}, TestPoint:TestPoint_Bridge_Pitch2.0mm_Drill0.7mm, F.Cu at (81.5, 52.0)
- added TP7: V_{E}, TestPoint:TestPoint_Bridge_Pitch2.0mm_Drill0.7mm, F.Cu at (81.5, 55.5)
- added TP8: V_{E}, TestPoint:TestPoint_Bridge_Pitch2.0mm_Drill0.7mm, F.Cu at (81.5, 58.9)
- added TP9: V_{SW}, TestPoint:TestPoint_Bridge_Pitch2.0mm_Drill0.7mm, F.Cu at (81.5, 62.4)
- added U1: MAX4073T, Package_TO_SOT_SMD:SOT-23-6_Handsoldering, F.Cu at (389.8, 99.9)
- added U10: ADS1014IDGS, Package_SO:TSSOP-10_3x3mm_P0.5mm, F.Cu at (217.3, 57.8)
- added U11: MC34063A, Package_SO:SOIC-8_3.9x4.9mm_P1.27mm, F.Cu at (109.1, 30.1)
- added U12: MC34063A, Package_SO:SOIC-8_3.9x4.9mm_P1.27mm, F.Cu at (109.1, 36.7)
- added U13: TPS54302, Package_TO_SOT_SMD:SOT-23-6_Handsoldering, F.Cu at (88.1, 58.8)
- added U14: LM74700, Package_TO_SOT_SMD:SOT-23-6_Handsoldering, F.Cu at (217.9, 174.5)
- added U15: BQ24640, ! Robomaster ICs:QFN50P350X350X100-17N-D, F.Cu at (243.5, 268.1)
- added U16: LM5123-Q1, Package_DFN_QFN:Texas_RGP0020H_VQFN-20-1EP_4x4mm_P0.5mm_EP2.4x2.4mm, F.Cu at (102.9, 257.6)
- added U17: TPS43061, ! Robomaster ICs:Texas_S-PWQFN-N16, F.Cu at (115.3, 138.4)
- added U18: TLV9301xDBV, Package_TO_SOT_SMD:SOT-23-5_HandSoldering, F.Cu at (345.1, 210.0)
- added U2: OPA551U, Package_SO:SOIC-8_3.9x4.9mm_P1.27mm, F.Cu at (385.3, 87.7)
- added U3: TLV9301xDBV, Package_TO_SOT_SMD:SOT-23-5_HandSoldering, F.Cu at (384.0, 99.9)
- added U4: OPA551U, Package_SO:SOIC-8_3.9x4.9mm_P1.27mm, F.Cu at (385.3, 94.2)
- added U5: TLV9301xDBV, Package_TO_SOT_SMD:SOT-23-5_HandSoldering, F.Cu at (384.0, 104.7)
- added U6: ISO164xB, Package_SO:SOIC-8_3.9x4.9mm_P1.27mm, F.Cu at (210.4, 66.7)
- added U7: ADS1014IDGS, Package_SO:TSSOP-10_3x3mm_P0.5mm, F.Cu at (217.3, 53.1)
- added U8: TLV9301xDBV, Package_TO_SOT_SMD:SOT-23-5_HandSoldering, F.Cu at (217.6, 65.8)
- added U9: DAC53401, Package_SON:WSON-8-1EP_2x2mm_P0.5mm_EP0.9x1.6mm, F.Cu at (216.9, 70.0)
Other:
- board text added: "Current Sense"
- board text added: "Dev Board Interface"
- board text added: "Housekeeping Power"
- board text added: "Ideal Diode"
- board text added: "Input Buck + Charger"
- board text added: "Output Boost 1"
- board text added: "Output Boost 2"
- board text added: "Supercap Host Board"

Commit message: Unsure of changes
Parts:
- C79, R70, R73, R74, U18: moved to B.Cu
- moved J30 250.8 mm to (273.8, 431.9)
- moved J31 250.8 mm to (273.8, 439.1)
- moved R75 250.8 mm to (285.4, 449.6)
- moved TP27 250.8 mm to (271.9, 451.4)
- moved TP28 250.8 mm to (271.9, 454.8)
- moved Q10 250.8 mm to (289.3, 432.4)
- moved R71 250.8 mm to (285.4, 446.3)
- moved R72 250.8 mm to (296.8, 437.0)
- moved TP25 250.8 mm to (271.9, 444.4)
- moved Q11 250.8 mm to (289.3, 440.6)
- moved TP26 250.8 mm to (271.9, 447.9)
- moved C74 243.9 mm to (324.1, 405.0)
- moved C75 243.4 mm to (324.1, 424.0)
- moved C78 229.6 mm to (336.8, 414.6), turned to 180 degrees
- moved C79 227.4 mm to (331.4, 414.4), turned to 90 degrees
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